Commit message: Baseline: sim launcher, colour-pick pick/place, sim perf and gripper fixes
Consolidates the outstanding work in the tree so later changes can be
reviewed against a clean mark.

arm_perception
- colour-pick now plays an ordered sequence per colour (shared pick, then an
  optional colour-specific place), chained from the motion-finished callback
  and abandoned if a step fails; new MotionStep domain value object.
- Recovery watchdog cancels and releases a motion that overruns, driven by a
  node timer so it fires even if the camera stalls; stale/duplicate completions
  are ignored.
- Config gained `place`/`place_duration_ms` with validation; malformed YAML is
  normalised to InvalidColorRangeError. Tests extended to cover all of it.

simulations
- Collision geometry: replaced detailed STL collision meshes with primitives
  where safe (arm links, shells, base, camera, imu), keeping meshes for the
  gripper assembly and mecanum wheels where the geometry matters. Collision
  triangles 21568 -> 7254.
- Gripper jaw links gained mu1/mu2 friction; they had none, so a gripped block
  slid straight out.
- colour_blocks_world: blocks shrunk to 3 cm and raised onto a low static shelf
  so the fixed pick pose can reach them.
- gazebo_arm/gazebo_moveit now default MACHINE_TYPE and LIDAR_TYPE like
  gazebo.launch.py did; without them xacro aborted and the launch died. Moved
  the defaults below the imports in all three, clearing the E402 lint.

File: src/simulations/jetrover_description/urdf/arm.urdf.xacro (robot description, xacro)
@@ -29,10 +29,7 @@
     </visual>
     <collision>
-      <origin
-        xyz="0 0 0"
-        rpy="0 0 0" />
-      <geometry>
-        <mesh
-          filename="package://jetrover_description/meshes/arm/link1.STL" />
+      <origin xyz="0.00006 0.00001 0.02114" rpy="0 0 0" />
+      <geometry>
+        <box size="0.04599 0.04602 0.04528" />
       </geometry>
     </collision>
@@ -65,10 +62,7 @@
     </visual>
     <collision>
-      <origin
-        xyz="0 0 0"
-        rpy="0 0 0" />
-      <geometry>
-        <mesh
-          filename="package://jetrover_description/meshes/arm/servo_link1_collision.stl" />
+      <origin xyz="0.00012 0.00240 0.02385" rpy="0 0 0" />
+      <geometry>
+        <box size="0.01924 0.04715 0.03923" />
       </geometry>
     </collision>
@@ -114,10 +108,7 @@
     </visual>
     <collision>
-      <origin
-        xyz="0 0 0"
-        rpy="0 0 0" />
-      <geometry>
-        <mesh
-          filename="package://jetrover_description/meshes/arm/link2_collision.stl" />
+      <origin xyz="0.00003 -0.00019 0.06571" rpy="0 0 0" />
+      <geometry>
+        <box size="0.03201 0.05600 0.16321" />
       </geometry>
     </collision>
@@ -168,10 +159,7 @@
     </visual>
     <collision>
-      <origin
-        xyz="0 0 0"
-        rpy="0 0 0" />
-      <geometry>
-        <mesh
-          filename="package://jetrover_description/meshes/arm/link3_collision.stl" />
+      <origin xyz="0.00000 -0.00050 0.06543" rpy="0 0 0" />
+      <geometry>
+        <box size="0.03201 0.05601 0.16324" />
       </geometry>
     </collision>
@@ -222,10 +210,7 @@
     </visual>
     <collision>
-      <origin
-        xyz="0 0 0"
-        rpy="0 0 0" />
-      <geometry>
-        <mesh
-          filename="package://jetrover_description/meshes/arm/link4_collision.stl" />
+      <origin xyz="0.00173 -0.00001 0.01903" rpy="0 0 0" />
+      <geometry>
+        <box size="0.04755 0.05602 0.07263" />
       </geometry>
     </collision>
@@ -276,10 +261,7 @@
     </visual>
     <collision>
-      <origin
-        xyz="0 0 0"
-        rpy="0 0 0" />
-      <geometry>
-        <mesh
-          filename="package://jetrover_description/meshes/arm/servo_link2_collision.stl" />
+      <origin xyz="0.00853 0.00001 -0.01405" rpy="0 0 0" />
+      <geometry>
+        <box size="0.03502 0.02604 0.02632" />
       </geometry>
     </collision>
@@ -325,10 +307,7 @@
     </visual>
     <collision>
-      <origin
-        xyz="0 0 0"
-        rpy="0 0 0" />
-      <geometry>
-        <mesh
-          filename="package://jetrover_description/meshes/arm/link5.STL" />
+      <origin xyz="-0.00005 -0.00002 0.00275" rpy="0 0 0" />
+      <geometry>
+        <box size="0.01904 0.01898 0.00550" />
       </geometry>
     </collision>

File: src/simulations/jetrover_description/urdf/car_mecanum.gazebo.urdf.xacro (robot description, xacro)
@@ -26,12 +26,9 @@
     </visual>
    <collision>
-      <origin
-        xyz="0 0 0"
-        rpy="0 0 0" />
-      <geometry>
-        <mesh
-          filename="package://jetrover_description/meshes/mecanum/base_link_collision.stl" />
-      </geometry>
-    </collision>
+     <origin xyz="-0.00083 -0.00000 -0.05640" rpy="0 0 0" />
+     <geometry>
+       <box size="0.30208 0.14567 0.05403" />
+     </geometry>
+   </collision>
   </link>
   <link

File: src/simulations/jetrover_description/urdf/car_mecanum.urdf.xacro (robot description, xacro)
@@ -26,12 +26,9 @@
     </visual>
    <collision>
-      <origin
-        xyz="0 0 0"
-        rpy="0 0 0" />
-      <geometry>
-        <mesh
-          filename="package://jetrover_description/meshes/mecanum/base_link_collision.stl" />
-      </geometry>
-    </collision>
+     <origin xyz="-0.00083 -0.00000 -0.05640" rpy="0 0 0" />
+     <geometry>
+       <box size="0.30208 0.14567 0.05403" />
+     </geometry>
+   </collision>
   </link>
   <link

File: src/simulations/jetrover_description/urdf/common.urdf.xacro (robot description, xacro)
@@ -28,10 +28,7 @@
     </visual>
     <collision>
-      <origin
-        xyz="0 0 0"
-        rpy="0 0 0" />
+      <origin xyz="-0.09927 -0.00018 0.07944" rpy="0 0 0" />
       <geometry>
-        <mesh
-          filename="package://jetrover_description/meshes/common/back_shell_black_link_collision.stl" />
+        <box size="0.12869 0.16530 0.15496" />
       </geometry>
     </collision>
@@ -77,10 +74,7 @@
     </visual>
     <collision>
-      <origin
-        xyz="0 0 0"
-        rpy="0 0 0" />
+      <origin xyz="-0.00326 -0.00017 0.01909" rpy="0 0 0" />
       <geometry>
-        <mesh
-          filename="package://jetrover_description/meshes/common/back_shell_green_link_collision.stl" />
+        <box size="0.30214 0.14402 0.11665" />
       </geometry>
     </collision>

File: src/simulations/jetrover_description/urdf/depth_camera.urdf.xacro (robot description, xacro)
@@ -29,10 +29,7 @@
     </visual>
     <collision>
-      <origin
-        xyz="0 0 0"
-        rpy="0 0 0" />
+      <origin xyz="-0.00051 0.01418 0.00138" rpy="0 0 0" />
       <geometry>
-        <mesh
-          filename="package://jetrover_description/meshes/arm/camera_connect_link.STL" />
+        <box size="0.05542 0.04494 0.00320" />
       </geometry>
     </collision>
@@ -82,10 +79,7 @@
     </visual>
     <collision>
-      <origin
-        xyz="0 0 0"
-        rpy="0 0 0" />
+      <origin xyz="0.00005 0.00079 -0.00001" rpy="0 0 0" />
       <geometry>
-        <mesh
-          filename="package://jetrover_description/meshes/arm/depth_cam_link_collision.stl" />
+        <box size="0.02488 0.09064 0.02514" />
       </geometry>
     </collision>

File: src/simulations/jetrover_description/urdf/gazebo.urdf.xacro (robot description, xacro)
@@ -66,5 +66,9 @@
       <update_rate>10</update_rate>
       <always_on>true</always_on>
-      <visualize>false</visualize>
+      <!-- Draws the scan rays inside Gazebo itself. On its own this only
+           marks the sensor as visualisable; the rays appear once the
+           VisualizeLidar GUI plugin is loaded, which the worlds' <gui>
+           block does. -->
+      <visualize>true</visualize>
       <lidar>
         <scan>

File: src/simulations/jetrover_description/urdf/gripper.urdf.xacro (robot description, xacro)
@@ -361,3 +361,21 @@
       offset="0" />
   </joint>
+  <!-- Grip friction. The jaw links had no surface friction, so even when the
+       fingers close on a block (mu 1.2, 50 g) it slid straight out. High mu on
+       the contacting jaw faces lets the closed gripper actually carry it.
+       NOTE: Gazebo friction grasping is force-sensitive - if a block still
+       slips after this, the grip force (r_joint closed target / effort) needs
+       tuning, or use a detachable-joint attacher. -->
+  <xacro:macro name="jaw_friction" params="link">
+    <gazebo reference="${link}">
+      <mu1>2.0</mu1>
+      <mu2>2.0</mu2>
+    </gazebo>
+  </xacro:macro>
+  <xacro:jaw_friction link="r_link"/>
+  <xacro:jaw_friction link="l_link"/>
+  <xacro:jaw_friction link="l_in_link"/>
+  <xacro:jaw_friction link="r_in_link"/>
+  <xacro:jaw_friction link="l_out_link"/>
+  <xacro:jaw_friction link="r_out_link"/>
 </robot>

File: src/simulations/jetrover_description/urdf/imu.urdf.xacro (robot description, xacro)
@@ -29,10 +29,7 @@
     </visual>
     <collision>
-      <origin
-        xyz="0 0 0"
-        rpy="0 0 0" />
+      <origin xyz="-0.01598 -0.01865 0.00080" rpy="0 0 0" />
       <geometry>
-        <mesh
-          filename="package://jetrover_description/meshes/common/imu_link.stl" />
+        <box size="0.06295 0.09000 0.00160" />
       </geometry>
     </collision>
